Commit message: 20220110: fin. urdf, strt. xacro

File: IMU_ws_mk2/LINES354_ws/src/test_pkg/urdf/demo_chp06_joint_robotCar.urdf (robot description, URDF)
Before this commit: robot mycar, 2 links, 1 joints
Links:
- added link base_footprint; visual sphere radius=0.001
Joints:
- added joint base_link2base_footprint: type fixed, parent base_footprint, child base_link, origin xyz=0 0 0.05
