Commit message: 20220110: fin. arbotix diff_controller

File: IMU_ws_mk2/LINES354_ws/src/test_pkg/urdf/xacro_myTurtleBot_arbotix/demo_chp06_myTurtleBot_chassis.xacro (robot description, xacro)
@@ -46,5 +46,6 @@
             </visual>
         </link>
-        <joint name="${name}_wheel2base_link" type="continuous">
+<!--        <joint name="${name}_wheel2base_link" type="continuous">-->
+        <joint name="base_${name}_wheel_joint" type="continuous">
             <parent link="base_link"/>
             <child link="${name}_wheel"/>
@@ -53,6 +54,8 @@
         </joint>
     </xacro:macro>
-    <xacro:add_wheel name="left" flag="1"/>
-    <xacro:add_wheel name="right" flag="-1"/>
+<!--    <xacro:add_wheel name="left" flag="1"/>-->
+<!--    <xacro:add_wheel name="right" flag="-1"/>-->
+    <xacro:add_wheel name="l" flag="1"/>
+    <xacro:add_wheel name="r" flag="-1"/>
     <!-- * * * * * * * * * universal wheels * * * * * * * * * -->
     <xacro:property name="universal_wheel_radius" value="0.0075"/>
