Commit message: 20220117: fin. chpt 0667: myTurtleBot with sim. sensors

File: IMU_ws_mk2/LINES354_ws/src/test_pkg/urdf/xacro_gazebo_bot_in_room/demo_chp066_myTurtleBot.xacro (robot description, xacro)
@@ -1,8 +1,4 @@
 <robot name="MyTurtleBot" xmlns:xacro="http://wiki.ros.org/xacro">
     <xacro:property name="file_path" value="$(find test_pkg)/urdf/xacro_gazebo_myTurtleBot"/>
-<!--    <xacro:include filename="${file_path}/demo_chp066_myTurtleBot_component.xacro" />-->
-<!--    <xacro:include filename="${file_path}/demo_chp066_myTurtleBot_chassis.xacro" />-->
-<!--    <xacro:include filename="${file_path}/demo_chp066_myTurtleBot_camera.xacro" />-->
-<!--    <xacro:include filename="${file_path}/demo_chp066_myTurtleBot_laser.xacro" />-->
     <xacro:include filename="$(find test_pkg)/urdf/xacro_gazebo_myTurtleBot/demo_chp066_myTurtleBot_component.xacro" />
     <xacro:include filename="$(find test_pkg)/urdf/xacro_gazebo_myTurtleBot/demo_chp066_myTurtleBot_chassis.xacro" />

File: IMU_ws_mk2/LINES354_ws/src/test_pkg/urdf/xacro_gazebo_chp0667_bot_sensors_room/myTurtleBot_laser.xacro (robot description, xacro)
@@ -1,9 +1,10 @@
 <robot name="MyTurtleBot_laser" xmlns:xacro="http://wiki.ros.org/xacro">
-    <!-- laser support frame property macro -->
     <xacro:property name="support_length" value="0.15"/>
     <xacro:property name="support_radius" value="0.01"/>
     <xacro:property name="support_x" value="0.0"/>
     <xacro:property name="support_y" value="0.0"/>
-    <xacro:property name="support_z" value="${base_link_length / 2 + support_length / 2}"/>
+    <xacro:property name="support_z"
+                    value="${base_link_length / 2 + support_length / 2}"/>
+    <xacro:property name="support_m" value="0.02"/>
     <link name="support">
         <visual>
@@ -16,4 +17,11 @@
             </material>
         </visual>
+        <collision>
+            <geometry>
+                <cylinder radius="${support_radius}" length="${support_length}"/>
+            </geometry>
+            <origin xyz="0.0 0.0 0.0" rpy="0.0 0.0 0.0"/>
+        </collision>
+        <xacro:cylinder_inertial_matrix m="${support_m}" r="${support_radius}" h="${support_length}"/>
     </link>
     <joint name="support2base_link" type="fixed">
@@ -22,10 +30,14 @@
         <origin xyz="${support_x} ${support_y} ${support_z}"/>
     </joint>
-    <!-- laser property macro -->
+    <gazebo reference="support">
+        <material>Gazebo/White</material>
+    </gazebo>
     <xacro:property name="laser_length" value="0.05"/>
     <xacro:property name="laser_radius" value="0.03"/>
     <xacro:property name="laser_x" value="0.0"/>
     <xacro:property name="laser_y" value="0.0"/>
-    <xacro:property name="laser_z" value="${support_length / 2 + laser_length / 2}"/>
+    <xacro:property name="laser_z"
+                    value="${support_length / 2 + laser_length / 2}"/>
+    <xacro:property name="laser_m" value="0.1"/>
     <link name="laser">
         <visual>
@@ -36,4 +48,11 @@
             <material name="black"/>
         </visual>
+        <collision>
+            <geometry>
+                <cylinder radius="${laser_radius}" length="${laser_length}"/>
+            </geometry>
+            <origin xyz="0.0 0.0 0.0" rpy="0.0 0.0 0.0"/>
+        </collision>
+        <xacro:cylinder_inertial_matrix m="${laser_m}" r="${laser_radius}" h="${laser_length}"/>
     </link>
     <joint name="laser2support" type="fixed">
@@ -42,3 +61,6 @@
         <origin xyz="${laser_x} ${laser_y} ${laser_z}"/>
     </joint>
+    <gazebo reference="laser">
+        <material>Gazebo/Black</material>
+    </gazebo>
 </robot>
